File: hardware/KiCad_new/_restore_backup_2026-07-08T14-49-28-121/KiCad_new.kicad_sch (KiCad schematic)
At the start: 20 parts, among them J102 Conn_01x02, J103 Conn_01x03, J104 Conn_01x08, J105 Conn_01x02, K101 G5LE-1, K102 G5LE-1, K103 G5LE-1, K104 G5LE-1, M101 AC Gear Motor, SW101 SW_DPST_x2, SW102 SW_DPST_x2, SW103 SW_DPST_x2

Commit message: Create PCB
Changed lines of the file:
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@@
+	(wire
+		(pts
+			(xy 236.22 125.73) (xy 237.49 125.73)
+		)
+		(stroke
+			(width 0)
+			(type default)
+		)
+	)
 	(wire
 		(pts
@@
 	(symbol
 		(lib_id "power:PWR_FLAG")
-		(at 237.49 125.73 90)
+		(at 236.22 125.73 90)
 		(unit 1)
 		(body_style 1)
@@
 		(fields_autoplaced yes)
 		(property "Reference" "#FLG0102"
-			(at 235.585 125.73 0)
+			(at 234.315 125.73 0)
 			(hide yes)
 			(show_name no)
@@
 		)
 		(property "Value" "PWR_FLAG"
-			(at 233.68 125.7299 90)
+			(at 232.41 125.7299 90)
 			(hide yes)
 			(show_name no)
@@
 		)
 		(property "Footprint" ""
-			(at 237.49 125.73 0)
+			(at 236.22 125.73 0)
 			(hide yes)
 			(show_name no)
@@
 		)
 		(property "Datasheet" ""
-			(at 237.49 125.73 0)
+			(at 236.22 125.73 0)
 			(hide yes)
 			(show_name no)
@@
 		)
 		(property "Description" "Special symbol for telling ERC where power comes from"
-			(at 237.49 125.73 0)
-			(hide yes)
-			(show_name no)
+			(at 236.22 125.73 0)
+			(hide yes)
+			(show_name no)
